File: 2025中/BALL Sensor/BALL Sensor V1.1/BALL Sensor V1.1.kicad_pcb (KiCad board)
At the start: 2 copper layers, 100 x 100 mm, 43 parts, among them J1 Conn_02x04_Odd_Even, J2 Conn_01x05_Pin, SW2 SW_MEC_5G, U2 ATmega32U4-A, Y1 CSTCE16M0V53-R0

Commit message: 定期更新
Routing:
- net +5V: track 378.5 -> 375.2 mm

Commit message: 定期更新
Parts:
- added R1: 10k, Resistor_SMD:R_0603_1608Metric, B.Cu at (128.0, 70.8)
- H1, H2, H3, H4: value MountingHole_3.2mm_M3 -> MountingHole
Connections:
- U2 pad 33: unconnected-(U2-~{HWB}/PE2-Pad33) -> Net-(U2-~{HWB}/PE2)
- U2 pad 42: +5V -> unconnected-(U2-AREF-Pad42)
Routing:
- net Net-(U2-~{HWB}/PE2): track 0.00 -> 2.19 mm, vias 0 -> 1
