File: 2025中/CATCH Sensor/LEDV1.1/LEDV1.1.kicad_pcb (KiCad board)
At the start: 2 copper layers, 6 x 12 mm, 3 parts, among them J1 Conn_01x02_Pin

Commit message: 定期更新
Other:
- board text added: "+"
- board text added: "-"
Changed lines of the file:
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@@
 			(psa4output no)
 			(plot_black_and_white yes)
-			(plotinvisibletext no)
 			(sketchpadsonfab no)
 			(plotpadnumbers no)
@@
 		(layer "Edge.Cuts")
 	)
+	(gr_text "-"
+		(at 149.4 103.99 0)
+		(layer "B.SilkS")
+		(effects
+			(font
+				(size 1 1)
+				(thickness 0.1)
+			)
+			(justify left bottom mirror)
+		)
+	)
+	(gr_text "+"
+		(at 152.02 103.99 0)
+		(layer "B.SilkS")
+		(effects
+			(font
+				(size 1 1)
+				(thickness 0.1)
+			)
+			(justify left bottom mirror)
+		)
+	)
 	(segment
