File: 2025中/MOTOR Driver/Motor Driver V1.1/Motor Driver V1.1.kicad_sch (KiCad schematic)
At the start: 46 parts, among them J1 Conn_01x08_Pin, J2 Conn_01x03_Pin, U1 DRV8874PWPR, U2 DRV8874PWPR, U3 DRV8874PWPR, U4 DRV8874PWPR

Commit message: 定期更新
Connections:
- net +3.3V: no longer U1.16 (PMODE), U2.16 (PMODE), U3.16 (PMODE), U4.16 (PMODE)
- net GND: now also U1.16 (PMODE), U2.16 (PMODE), U3.16 (PMODE), U4.16 (PMODE)
