File: 2025前/MAIN/MAIN V1.1/MAIN V1.1.kicad_sch (KiCad schematic)
At the start: 51 parts, among them U1 Mega 2560 ProMini footprint

Commit message: 定期更新
Changed lines of the file:
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@@
 (kicad_sch
-	(version 20231120)
+	(version 20250114)
 	(generator "eeschema")
-	(generator_version "8.0")
+	(generator_version "9.0")
 	(paper "A3")
 	(junction
@@
 		)
 	)
+	(embedded_fonts no)
 )
